File: LiPo_BuckBoost_Charger.kicad_pcb (KiCad board)
At the start: 4 copper layers, 53 x 33 mm, 63 parts, among them J1 Type-C_6P, J2 JST PH Connector, J3 Conn_01x01, J4 Conn_01x01, J5 JST PH Connector, J6 JST PH Connector, J7 JST PH Connector, Q1 SI2301, Q2 SI2301, U1 TP4056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

Commit message: updated version number on pcb, updated readme
Other:
- board text added: "Potpurri TP4056 LiPo Charger with TPS63020 Buck-Boost Converter Version 1.3"
- board text removed: "Potpurri TP4056 LiPo Charger with TPS63020 Buck-Boost Converter Version 1.2"
Changed lines of the file:
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@@
     (effects (font (size 0.8 0.8) (thickness 0.15) bold) (justify left bottom))
   )
-  (gr_text "Potpurri\nTP4056 LiPo Charger with\nTPS63020 Buck-Boost Converter\nVersion 1.2" (at 97.3328 54.3052) (layer "B.Mask")
+  (gr_text "Potpurri\nTP4056 LiPo Charger with\nTPS63020 Buck-Boost Converter\nVersion 1.3" (at 97.3328 54.3052) (layer "B.Mask")
     (effects (font (size 0.7 0.7) (thickness 0.15) bold) (justify left bottom mirror))
   )
